Commit message: fixed xacro missing namespace (depreciation warning)

File: kinect_description/urdf/stand/macros.xacro (robot description, xacro)
@@ -1,9 +1,9 @@
 <?xml version="1.0"?>
 <robot name="mybot" xmlns:xacro="http://www.ros.org/wiki/xacro">
-    <macro name="cylinder_inertia" params="m r h">
+    <xacro:macro name="cylinder_inertia" params="m r h">
         <inertia  ixx="${m*(3*r*r+h*h)/12}" ixy = "0" ixz = "0"
                   iyy="${m*(3*r*r+h*h)/12}" iyz = "0"
                   izz="${m*r*r/2}"
         />
-    </macro>
+    </xacro:macro>
 </robot>
